File: maincircuit/maincircuit.kicad_sch (KiCad schematic)
At the start: 0 parts

Commit message: [add]ControlCircuit完成
Other:
- sheet Emergency ports: added EMERGENCY, GNDPWR, LOAD, VCCPWR; removed none
Changed lines of the file:
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@@
+			)
+		)
+		(pin "EMERGENCY" input
+			(at 157.48 96.52 180)
+			(effects
+				(font
+					(size 1.27 1.27)
+				)
+				(justify left)
+			)
+		)
+		(pin "GNDPWR" output
+			(at 184.15 121.92 270)
+			(effects
+				(font
+					(size 1.27 1.27)
+				)
+				(justify left)
+			)
+		)
+		(pin "VCCPWR" input
+			(at 179.07 74.93 90)
+			(effects
+				(font
+					(size 1.27 1.27)
+				)
+				(justify right)
+			)
+		)
+		(pin "LOAD" input
+			(at 194.31 74.93 90)
+			(effects
+				(font
+					(size 1.27 1.27)
+				)
+				(justify right)
 			)
 		)
