File: maincircuit/ControlCircuit.kicad_pcb (KiCad board)
At the start: 4 copper layers, 60 x 80 mm, 96 parts, among them J1 USB_C_Receptacle_USB2.0_16P, J10 Conn_02x03_Odd_Even, J11 Conn_02x03_Odd_Even, J12 Conn_02x04_Odd_Even, J13 Conn_01x03_Pin, J14 Conn_01x02_Pin, J15 Conn_01x05_Pin, J16 Conn_01x02_Pin, J3 Conn_02x02_Counter_Clockwise, J4 Conn_01x06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

Commit message: add: ver1.0の基板データの完成
Other:
- board text added: "D"
- board text added: "JLCJLCJLC"
- board text added: "M1"
- board text added: "M2"
